File: UIAPduino-breakout-board.kicad_sch (KiCad schematic)
At the start: 13 parts, among them J1 Conn_01x20_Pin, J2 Conn_01x20_Socket, J3 Barrel_Jack_Switch, U3 L7805

Commit message: 修正
Connections:
- net +12V: no longer J3.3
- net GND: now also J3.3
Changed lines of the file:
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@@
-	)
-	(junction
-		(at 63.5 156.21)
-		(diameter 0)
-		(color 0 0 0 0)
 	)
 	(junction
@@
 	)
 	(junction
+		(at 63.5 161.29)
+		(diameter 0)
+		(color 0 0 0 0)
+	)
+	(junction
 		(at 205.74 76.2)
 		(diameter 0)
@@
 	(wire
 		(pts
+			(xy 63.5 158.75) (xy 63.5 161.29)
+		)
+		(stroke
+			(width 0)
+			(type default)
+		)
+	)
+	(wire
+		(pts
 			(xy 130.81 104.14) (xy 213.36 104.14)
 		)
@@
 		)
 		(stroke
-			(width 0)
-			(type default)
-		)
-	)
-	(wire
-		(pts
-			(xy 63.5 158.75) (xy 63.5 156.21)
-		)
-		(stroke
